Commit message: Update m2wr_description

File: m2wr_description/urdf/m2wr.xacro (robot description, xacro)
@@ -2,7 +2,8 @@
 <!-- Declare the robot name -->
 <robot xmlns:xacro="http://www.ros.org/wiki/xacro" name="m2wr">
-  <!-- Include other xacro files-->
+  <!-- Import all Gazebo-customization elements, including Gazebo colors -->
+  <xacro:include filename="$(find m2wr_description)/urdf/m2wr.gazebo" />
+  <!-- Import Rviz colors -->
   <xacro:include filename="$(find m2wr_description)/urdf/materials.xacro" />
-  <xacro:include filename="$(find m2wr_description)/urdf/m2wr.gazebo" />
   <xacro:include filename="$(find m2wr_description)/urdf/macros.xacro" />
   <!-- Define chassis link of the robot, the base_link -->
@@ -162,3 +163,23 @@
   </joint>
   -->
+  <transmission name="tran1">
+    <type>transmission_interface/SimpleTransmission</type>
+    <joint name="joint_right_wheel">
+      <hardwareInterface>hardware_interface/EffortJointInterface</hardwareInterface>
+    </joint>
+    <actuator name="motor1">
+      <hardwareInterface>hardware_interface/EffortJointInterface</hardwareInterface>
+      <mechanicalReduction>1</mechanicalReduction>
+    </actuator>
+  </transmission>
+  <transmission name="tran2">
+    <type>transmission_interface/SimpleTransmission</type>
+    <joint name="joint_left_wheel">
+      <hardwareInterface>hardware_interface/EffortJointInterface</hardwareInterface>
+    </joint>
+    <actuator name="motor2">
+      <hardwareInterface>hardware_interface/EffortJointInterface</hardwareInterface>
+      <mechanicalReduction>1</mechanicalReduction>
+    </actuator>
+  </transmission>
 </robot>

File: m2wr_description/urdf/materials.xacro (robot description, xacro)
@@ -6,20 +6,20 @@
   </material>
   <material name="blue">
-      <color rgba="0 0 1.0 1.0"/>
+      <color rgba="0 0 0.8 1.0"/>
   </material>
   <material name="green">
-      <color rgba="0.0 1.0 0.0 1.0"/>
+      <color rgba="0.0 0.8 0.0 1.0"/>
   </material>
   <material name="grey">
-      <color rgba="0.5 0.5 0.5 1.0"/>
+      <color rgba="0.2 0.2 0.2 1.0"/>
   </material>
   <material name="orange">
-      <color rgba="1.0 0.423529411765 0.0392156862745 1.0"/>
+      <color rgba="${255/255} ${108/255} ${10/255} 1.0"/>
   </material>
   <material name="brown">
-      <color rgba="0.870588235294 0.811764705882 0.764705882353 1.0"/>
+      <color rgba="${222/255} ${207/255} ${195/255} 1.0"/>
   </material>
   <material name="red">
-      <color rgba="0.80078125 0.12890625 0.1328125 1.0"/>
+      <color rgba="0.8 0.0 0.0 1.0"/>
   </material>
   <material name="white">
